Commit message: FIX Now loads custom quadrotor configuration
In the earlier commit, the main launch file did not use the custom
quadrotor configuration supplied with the project.

When the quadrotor was added, the launch file crashed with a
"quadrotor_plugins" macro not found exception.

A similar exception occured here: https://github.com/tu-darmstadt-ros-pkg/hector_quadrotor/issues/37
On that basis, I have surrounded the quadrotor_plugins.xacro
inclusion with the appropriate tags in quadrotor_configuration.gazebo.xacro.
Roslaunch now appears to work correctly.

File: pprz_ros_template_project/urdf/configuration/quadrotor_configuration.gazebo.xacro (robot description, xacro)
@@ -2,5 +2,7 @@
 <robot name="quadrotor" xmlns:xacro="http://www.ros.org/wiki/xacro">
     <xacro:include filename="$(find pprz_ros_template_project)/urdf/configuration/quadrotor_configuration.urdf.xacro" /><!-- configuration URDF file -->
-    <xacro:include filename="$(find hector_quadrotor_gazebo)/urdf/quadrotor_plugins.gazebo.xacro" />
+    <xacro:macro name="quadrotor_plugins"><!-- FIX missing quadrotor_plugins macro -->
+    	<xacro:include filename="$(find hector_quadrotor_gazebo)/urdf/quadrotor_plugins.gazebo.xacro" />
+    </xacro:macro>
     <xacro:quadrotor_plugins />
 </robot>
